File: Hardware/Lora TDS sensor V1.2.sch (EAGLE design)
At the start: 103 parts, among them J5 PH2.0-2P-90-DIP, Q1 MOSFET-PCHANNEL, Q2 AO3400, Q3 MOSFET-PCHANNEL, U1 1117/3V3, U2 ATMEGA328P, U3 LM324_1, U4 RFM95_98W, U5 XC6206P302, U6 TP4056, U7 CD4060, U8 TPS60400DBVR, U9 DW06D, Y1 CSTCE16M0V53-R0 8MHZ

Commit message: Update V1.2
Parts:
- removed D3: 0R, adafruit:DIODESOD-323F
- removed J3: (no value), Connector:HEADER-3P-2.54
- removed PWR: red, Discrete:LED'0603'
- removed R22: 10k, Discrete:R-0603
- removed R39: NC, Discrete:R-0603
- removed U5: XC6206P302, 1mytest:XC6206P302
- added C11: 10uF/NC, Discrete:C-0603
- added C16: 10uF, Discrete:C-0603
- added C28: 0.1uF, Discrete:C-0603
- added C29, C33: 100nF, Discrete:C-0603
- added C32, C34: 4.7uF, Discrete:C-0603
- added C35: NC, Discrete:C-0603
- added J6: (no value), Connector-new:GROVE-CONNECTOR-SMD'90D'
- added R44: NC, Discrete:R-0603
- C26: value 10uF -> 100nF
- C27: value 4.7uF -> NC
- R1: value NC -> 0R
- R15: value 10k -> 10K
- R27: value 1M -> 340K
- R36: value 330R -> 1K
- U1: value 1117/3V3 -> SPX3819; device IC:LD1117'SOT89' -> IC:SPX3819
Connections:
- new net NC: J6.2
- net +3V0: now also C11.2, C28.2, C29.1, C34.2, C35.2, R44.2, U1.VOUT; no longer C25.2, R39.2, U5.VOUT
- net -3V0: now also C25.1, C32.2, C33.2
- net A1: now also J6.1, R37.1; no longer J3.P$3, R37.2
- net A4/SDA: no longer R15.2
- net A5/SCL: no longer R22.2
- net D5: no longer R38.2
- net GND: now also C11.1, C16.1, C25.2, C28.1, C29.2, C32.1, C33.1, C34.1, C35.1, J6.4, J6.SS1, J6.SS2, R38.2; no longer C25.1, J3.P$2, R36.2, U5.VSS
- net N$2: now also R36.2, U1.EN; no longer D3.C, R1.2, U1.IN
- net N$7: now also Q1.G, R15.2; no longer PWR.-, R36.1
- net N$8: now also R15.1; no longer Q1.G
- net VCC: now also C16.2, J6.3, LED.+, R36.1, R37.2, R44.1, U1.VIN; no longer J3.P$1, R37.1, R39.1, U5.VIN
- net VDD: no longer LED.+, PWR.+, R15.1, R22.1, U1.OUT
- net VIN: now also R1.2; no longer D3.A
Other:
- note added: "3V to -3V"
- note added: "Charger"
- note added: "DS18B20 Interface"
- note added: "LoRa-TDS sensor V1.2"
- note added: "Protect"
- note added: "TDS Detect"
- note added: "VDD to 3V"
- note removed: "+3V"
- note removed: "+3V3"
- note removed: "+5V"
- note removed: "-3V"
- note removed: "1.8v-3.7v"
- note removed: "1.8v-5.5v"
- note removed: "2-pin interface"
- note removed: "3-pin interface"
- note removed: "328P"
- note removed: "40mA"
- note removed: "A0"
- note removed: "A1"
- note removed: "AAA 2.5-3v"
- note removed: "Battery"
- note removed: "CD4060"
- note removed: "CD4060+LM324"
- note removed: "CP2104"
- note removed: "Charge"
- note removed: "LDO&Charger"
- note removed: "Li 3v-4.3v(3.7V)"
- note removed: "LoRa TDS sensor"
- note removed: "LoRa-TDS sensor V1.1"
- note removed: "SPI"
- note removed: "TDS"
- note removed: "TEMP"
- note removed: "TP4056"
- note removed: "USB"
- note removed: "converter"
- moved on the sheet: C18, C2, C25, C26, C27, C30, C31, C5, C6, D1, D4, D8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
